File: pcb_files/pcb_design/pcb_design.kicad_pcb (KiCad board)
At the start: 2 copper layers, 109.2 x 83.8 mm, 6 parts, among them J1 Screw_Terminal_01x02, U5 Pico

Commit message: updated pcb files
Connections:
- U5 pad 21: Net-(U2-TXD) -> Net-(U2-RXD)
- U5 pad 22: Net-(U2-RXD) -> Net-(U2-TXD)
Routing:
- net Net-(U2-RXD): track 80.0 -> 110.3 mm
Changed lines of the file:
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@@
       (net 21 "Net-(U4-MOSI)") (pinfunction "GPIO15") (pintype "bidirectional"))
     (pad "21" thru_hole oval (at 8.89 24.13) (size 1.7 1.7) (drill 1.02) (layers "*.Cu" "*.Mask")
-      (net 13 "Net-(U2-TXD)") (pinfunction "GPIO16") (pintype "bidirectional"))
+      (net 12 "Net-(U2-RXD)") (pinfunction "GPIO16") (pintype "bidirectional"))
     (pad "21" smd rect (at 8.89 24.13) (size 3.5 1.7) (drill (offset 0.9 0)) (layers "F.Cu" "F.Mask")
-      (net 13 "Net-(U2-TXD)") (pinfunction "GPIO16") (pintype "bidirectional"))
+      (net 12 "Net-(U2-RXD)") (pinfunction "GPIO16") (pintype "bidirectional"))
     (pad "22" thru_hole oval (at 8.89 21.59) (size 1.7 1.7) (drill 1.02) (layers "*.Cu" "*.Mask")
-      (net 12 "Net-(U2-RXD)") (pinfunction "GPIO17") (pintype "bidirectional"))
+      (net 13 "Net-(U2-TXD)") (pinfunction "GPIO17") (pintype "bidirectional"))
     (pad "22" smd rect (at 8.89 21.59) (size 3.5 1.7) (drill (offset 0.9 0)) (layers "F.Cu" "F.Mask")
-      (net 12 "Net-(U2-RXD)") (pinfunction "GPIO17") (pintype "bidirectional"))
+      (net 13 "Net-(U2-TXD)") (pinfunction "GPIO17") (pintype "bidirectional"))
     (pad "23" thru_hole rect (at 8.89 19.05) (size 1.7 1.7) (drill 1.02) (layers "*.Cu" "*.Mask")
       (net 11 "Net-(U2-GND)") (pinfunction "GND") (pintype "power_in"))
@@
   (segment (start 165.1 48.26) (end 165.1 109.22) (width 0.25) (layer "F.Cu") (net 11))
   (segment (start 162.56 45.72) (end 165.1 48.26) (width 0.25) (layer "F.Cu") (net 11))
-  (segment (start 165.1 53.34) (end 177.8 66.04) (width 0.25) (layer "B.Cu") (net 12))
-  (segment (start 177.8 66.04) (end 177.8 109.22) (width 0.25) (layer "B.Cu") (net 12))
-  (segment (start 177.8 109.22) (end 175.26 111.76) (width 0.25) (layer "B.Cu") (net 12))
-  (segment (start 175.26 111.76) (end 167.64 111.76) (width 0.25) (layer "B.Cu") (net 12))
-  (segment (start 165.1 45.72) (end 165.1 53.34) (width 0.25) (layer "B.Cu") (net 12))
-  (segment (start 180.34 109.22) (end 175.26 114.3) (width 0.25) (layer "B.Cu") (net 13))
+  (segment (start 185.42 43.18) (end 185.42 111.76) (width 0.25) (layer "B.Cu") (net 12))
+  (segment (start 185.42 111.76) (end 182.88 114.3) (width 0.25) (layer "B.Cu") (net 12))
+  (segment (start 165.1 45.72) (end 165.1 43.18) (width 0.25) (layer "B.Cu") (net 12))
+  (segment (start 165.1 43.18) (end 185.42 43.18) (width 0.25) (layer "B.Cu") (net 12))
+  (segment (start 182.88 114.3) (end 167.64 114.3) (width 0.25) (layer "B.Cu") (net 12))
   (segment (start 167.64 45.72) (end 180.34 58.42) (width 0.25) (layer "B.Cu") (net 13))
+  (segment (start 180.34 109.22) (end 180.34 111.76) (width 0.25) (layer "B.Cu") (net 13))
   (segment (start 180.34 58.42) (end 180.34 109.22) (width 0.25) (layer "B.Cu") (net 13))
-  (segment (start 175.26 114.3) (end 167.64 114.3) (width 0.25) (layer "B.Cu") (net 13))
+  (segment (start 180.34 111.76) (end 167.64 111.76) (width 0.25) (layer "B.Cu") (net 13))
   (segment (start 132.08 78.74) (end 134.62 81.28) (width 0.25) (layer "B.Cu") (net 16))
   (segment (start 132.08 45.72) (end 132.08 78.74) (width 0.25) (layer "B.Cu") (net 16))
