File: pcb_files/pcb_design/pcb_design.kicad_sch (KiCad schematic)
At the start: 6 parts, among them J1 Screw_Terminal_01x02, U5 Pico

Commit message: updated pcb files
Connections:
- net at U2.3 (RXD): now also U5.21 (GPIO16); no longer U5.22 (GPIO17)
- net at U2.4 (TXD): now also U5.22 (GPIO17); no longer U5.21 (GPIO16)
Changed lines of the file:
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@@
-    (stroke (width 0) (type default))
-  )
-  (wire (pts (xy 171.45 140.97) (xy 162.56 140.97))
     (stroke (width 0) (type default))
   )
@@
     (stroke (width 0) (type default))
   )
-  (wire (pts (xy 171.45 77.47) (xy 171.45 140.97))
-    (stroke (width 0) (type default))
-  )
   (wire (pts (xy 163.83 90.17) (xy 163.83 97.79))
     (stroke (width 0) (type default))
@@
     (stroke (width 0) (type default))
   )
-  (wire (pts (xy 173.99 143.51) (xy 162.56 143.51))
-    (stroke (width 0) (type default))
-  )
   (wire (pts (xy 142.24 76.2) (xy 142.24 78.74))
     (stroke (width 0) (type default))
@@
     (stroke (width 0) (type default))
   )
+  (wire (pts (xy 171.45 143.51) (xy 162.56 143.51))
+    (stroke (width 0) (type default))
+  )
+  (wire (pts (xy 173.99 140.97) (xy 173.99 77.47))
+    (stroke (width 0) (type default))
+  )
   (wire (pts (xy 119.38 73.66) (xy 119.38 110.49))
+    (stroke (width 0) (type default))
+  )
+  (wire (pts (xy 162.56 140.97) (xy 173.99 140.97))
     (stroke (width 0) (type default))
   )
@@
     (stroke (width 0) (type default))
   )
-  (wire (pts (xy 173.99 77.47) (xy 173.99 143.51))
+  (wire (pts (xy 171.45 77.47) (xy 171.45 143.51))
     (stroke (width 0) (type default))
   )
